File: kp3sExpander.kicad_pcb (KiCad board)
At the start: 2 copper layers, 80 x 50 mm, 8 parts, among them J1 Conn_01x32_Female, J2 Conn_02x14_Odd_Even, J3 Conn_02x06_Odd_Even, J4 Conn_02x06_Odd_Even

Commit message: finalize v0.1
Parts:
- H1, H2, H3, H4: footprint MountingHole:MountingHole_3.2mm_M3 -> MountingHole:MountingHole_3.2mm_M3_DIN965_Pad
- J1: value Conn_01x32_Female -> Conn_01x33_Female
- moved J1 0.10 mm to (153.6, 74.7)
Routing:
- net GND: track 42.4 -> 55.1 mm, vias 0 -> 7
- net VCC: track 45.6 -> 58.2 mm
- net (no net): track 0.00 -> 10.4 mm
- net PD9: track 36.9 -> 31.9 mm
- net INT: track 60.6 -> 56.6 mm
- added copper zone on B.Cu, net GND
- added copper zone on F.Cu, net GND
Other:
- outline, holes or cut-outs redrawn
- board text added: "JLCJLCJLCJLC"
- board text added: "robin_nano-GPIO-expander v0.1 9R 2022"
