File: kp3sExpander.kicad_sch (KiCad schematic)
At the start: 8 parts, among them J1 Conn_01x32_Female, J2 Conn_02x14_Odd_Even, J3 Conn_02x06_Odd_Even, J4 Conn_02x06_Odd_Even

Commit message: finalize v0.1
Parts:
- removed J1: Conn_01x32_Female, kp3sExpander:FPC_32, symbol Connector:Conn_01x32_Female
- added J1: Conn_01x33_Female, kp3sExpander:FPC_32, symbol Connector:Conn_01x33_Female
- H1, H2, H3, H4: footprint MountingHole:MountingHole_3.2mm_M3 -> MountingHole:MountingHole_3.2mm_M3_DIN965_Pad
Connections:
- net +3V3: now also J1.1 (Pin_1)
- net GND: now also J1.2 (Pin_2), J1.32 (Pin_32), J1.33 (Pin_33)
- net INT: now also J1.26 (Pin_26)
- net PC5_BEEPER: now also J1.28 (Pin_28)
- net PC6: now also J1.23 (Pin_23)
- net PD0: now also J1.5 (Pin_5)
- net PD1: now also J1.6 (Pin_6)
- net PD10: now also J1.18 (Pin_18)
- net PD11: now also J1.20 (Pin_20)
- net PD13: now also J1.24 (Pin_24)
- net PD14: now also J1.3 (Pin_3)
- net PD15: now also J1.4 (Pin_4)
- net PD4: now also J1.22 (Pin_22)
- net PD5: now also J1.21 (Pin_21)
- net PD7: now also J1.19 (Pin_19)
- net PD8: now also J1.16 (Pin_16)
- net PD9: now also J1.17 (Pin_17)
- net PE10: now also J1.10 (Pin_10)
- net PE11: now also J1.11 (Pin_11)
- net PE12: now also J1.12 (Pin_12)
- net PE13: now also J1.13 (Pin_13)
- net PE14: now also J1.14 (Pin_14)
- net PE15: now also J1.15 (Pin_15)
- net PE7: now also J1.7 (Pin_7)
- net PE8: now also J1.8 (Pin_8)
- net PE9: now also J1.9 (Pin_9)
- net SPI2_MISO: now also J1.25 (Pin_25)
- net SPI2_MOSI: now also J1.27 (Pin_27)
- net SPI2_NSS: now also J1.31 (Pin_31)
- net SPI2_SCK: now also J1.29 (Pin_29)
- net VCC: now also J1.30 (Pin_30)
Changed lines of the file:
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@@
+    (stroke (width 0) (type default) (color 0 0 0 0))
+  )
+  (wire (pts (xy 92.71 36.83) (xy 92.71 39.37))
     (stroke (width 0) (type default) (color 0 0 0 0))
   )
@@
       (effects (font (size 1.27 1.27)) (justify left) hide)
     )
-  )
-  (symbol (lib_id "Connector:Conn_01x32_Female") (at 87.63 80.01 180) (unit 1)
-    (in_bom yes) (on_board yes)
-    (property "Reference" "J1" (id 0) (at 90.3732 33.655 0))
-    (property "Value" "Conn_01x32_Female" (id 1) (at 90.3732 35.9664 0))
-    (property "Footprint" "kp3sExpander:FPC_32" (id 2) (at 87.63 80.01 0)
-      (effects (font (size 1.27 1.27)) hide)
-    )
-    (property "Datasheet" "~" (id 3) (at 87.63 80.01 0)
-      (effects (font (size 1.27 1.27)) hide)
-    )
-    (pin "1")
-    (pin "10")
-    (pin "11")
-    (pin "12")
-    (pin "13")
-    (pin "14")
-    (pin "15")
-    (pin "16")
-    (pin "17")
-    (pin "18")
-    (pin "19")
-    (pin "2")
-    (pin "20")
-    (pin "21")
-    (pin "22")
-    (pin "23")
-    (pin "24")
-    (pin "25")
-    (pin "26")
-    (pin "27")
-    (pin "28")
-    (pin "29")
-    (pin "3")
-    (pin "30")
-    (pin "31")
-    (pin "32")
-    (pin "4")
-    (pin "5")
-    (pin "6")
-    (pin "7")
-    (pin "8")
-    (pin "9")
   )
   (symbol (lib_id "Connector_Generic:Conn_02x06_Odd_Even") (at 148.59 86.36 0) (unit 1)
@@
       (effects (font (size 1.27 1.27)) (justify left))
     )
-    (property "Footprint" "MountingHole:MountingHole_3.2mm_M3" (id 2) (at 185.42 43.18 0)
+    (property "Footprint" "MountingHole:MountingHole_3.2mm_M3_DIN965_Pad" (id 2) (at 185.42 43.18 0)
       (effects (font (size 1.27 1.27)) hide)
     )
@@
       (effects (font (size 1.27 1.27)) (justify left))
     )
-    (property "Footprint" "MountingHole:MountingHole_3.2mm_M3" (id 2) (at 185.42 55.88 0)
+    (property "Footprint" "MountingHole:MountingHole_3.2mm_M3_DIN965_Pad" (id 2) (at 185.42 55.88 0)
       (effects (font (size 1.27 1.27)) hide)
     )
@@
       (effects (font (size 1.27 1.27)) (justify left))
     )
-    (property "Footprint" "MountingHole:MountingHole_3.2mm_M3" (id 2) (at 185.42 49.53 0)
+    (property "Footprint" "MountingHole:MountingHole_3.2mm_M3_DIN965_Pad" (id 2) (at 185.42 49.53 0)
       (effects (font (size 1.27 1.27)) hide)
     )
@@
       (effects (font (size 1.27 1.27)) (justify left))
     )
-    (property "Footprint" "MountingHole:MountingHole_3.2mm_M3" (id 2) (at 185.42 36.83 0)
+    (property "Footprint" "MountingHole:MountingHole_3.2mm_M3_DIN965_Pad" (id 2) (at 185.42 36.83 0)
       (effects (font (size 1.27 1.27)) hide)
     )
@@
     )
     (pin "1")
+  )
+  (symbol (lib_id "Connector:Conn_01x33_Female") (at 87.63 77.47 180) (unit 1)
+    (in_bom yes) (on_board yes)
+    (property "Reference" "J1" (id 0) (at 85.09 36.83 0))
+    (property "Value" "Conn_01x33_Female" (id 1) (at 85.09 109.22 90))
+    (property "Footprint" "kp3sExpander:FPC_32" (id 2) (at 87.63 77.47 0)
+      (effects (font (size 1.27 1.27)) hide)
+    )
+    (property "Datasheet" "~" (id 3) (at 87.63 77.47 0)
+      (effects (font (size 1.27 1.27)) hide)
+    )
+    (pin "1")
+    (pin "10")
+    (pin "11")
+    (pin "12")
+    (pin "13")
+    (pin "14")
+    (pin "15")
+    (pin "16")
+    (pin "17")
+    (pin "18")
+    (pin "19")
+    (pin "2")
+    (pin "20")
+    (pin "21")
+    (pin "22")
+    (pin "23")
+    (pin "24")
+    (pin "25")
+    (pin "26")
+    (pin "27")
+    (pin "28")
+    (pin "29")
+    (pin "3")
+    (pin "30")
+    (pin "31")
+    (pin "32")
+    (pin "33")
+    (pin "4")
+    (pin "5")
+    (pin "6")
+    (pin "7")
+    (pin "8")
+    (pin "9")
   )
   (symbol (lib_id "power:+3V3") (at 50.8 43.18 0) (unit 1)
@@
     )
     (path "/78eb5c71-593e-4b7d-aeee-72127c3da07e"
-      (reference "H1") (unit 1) (value "MountingHole") (footprint "MountingHole:MountingHole_3.2mm_M3")
+      (reference "H1") (unit 1) (value "MountingHole") (footprint "MountingHole:MountingHole_3.2mm_M3_DIN965_Pad")
     )
     (path "/399d85f6-cd8f-492c-9c61-92929c7b03e3"
-      (reference "H2") (unit 1) (value "MountingHole") (footprint "MountingHole:MountingHole_3.2mm_M3")
+      (reference "H2") (unit 1) (value "MountingHole") (footprint "MountingHole:MountingHole_3.2mm_M3_DIN965_Pad")
     )
     (path "/5f502b09-63cb-46ac-a803-a353adca1ad9"
-      (reference "H3") (unit 1) (value "MountingHole") (footprint "MountingHole:MountingHole_3.2mm_M3")
+      (reference "H3") (unit 1) (value "MountingHole") (footprint "MountingHole:MountingHole_3.2mm_M3_DIN965_Pad")
     )
     (path "/41fc605d-4371-4fc8-ab4d-ee3bb0a68876"
-      (reference "H4") (unit 1) (value "MountingHole") (footprint "MountingHole:MountingHole_3.2mm_M3")
-    )
-    (path "/00000000-0000-0000-0000-000061d38b4d"
-      (reference "J1") (unit 1) (value "Conn_01x32_Female") (footprint "kp3sExpander:FPC_32")
+      (reference "H4") (unit 1) (value "MountingHole") (footprint "MountingHole:MountingHole_3.2mm_M3_DIN965_Pad")
+    )
+    (path "/9be71b4b-976f-45e7-97ed-42fe4498c1b0"
+      (reference "J1") (unit 1) (value "Conn_01x33_Female") (footprint "kp3sExpander:FPC_32")
     )
     (path "/462c89bc-d84c-443d-9798-5f65e0963468"
